Commit message: Update 2F-85 to reflect hardware version 4
Slight geometry changes to every part of the gripper, so all meshes replaced with new ones made from the latest CAD files
Adopt Robotiq's names for the components for consistency
Update to latest eSeries coupling hardware
Note hardware version in the readme so future users don't get confused like we did
Bump CMake min versions to silence warnings in noetic

File: robotiq_2f_85_gripper_gazebo/urdf/robotiq_arg2f_85_macro.xacro (robot description, xacro)
@@ -30,20 +30,20 @@
       <plugin filename="libroboticsgroup_upatras_gazebo_mimic_joint_plugin.so" name="${prefix}mimic_robotiq_85_1">
         <joint>${prefix}finger_joint</joint>
-        <mimicJoint>${prefix}left_inner_knuckle_joint</mimicJoint>
+        <mimicJoint>${prefix}left_proximal_phalanx_joint</mimicJoint>
         <multiplier>1.0</multiplier>
       </plugin>
       <plugin filename="libroboticsgroup_upatras_gazebo_mimic_joint_plugin.so" name="${prefix}mimic_robotiq_85_2">
         <joint>${prefix}finger_joint</joint>
-        <mimicJoint>${prefix}left_inner_finger_joint</mimicJoint>
+        <mimicJoint>${prefix}left_distal_phalanx_joint</mimicJoint>
         <multiplier>-1.0</multiplier>
       </plugin>
       <plugin filename="libroboticsgroup_upatras_gazebo_mimic_joint_plugin.so" name="${prefix}mimic_robotiq_85_3">
         <joint>${prefix}finger_joint</joint>
-        <mimicJoint>${prefix}right_inner_knuckle_joint</mimicJoint>
+        <mimicJoint>${prefix}right_proximal_phalanx_joint</mimicJoint>
         <multiplier>1.0</multiplier>
       </plugin>
       <plugin filename="libroboticsgroup_upatras_gazebo_mimic_joint_plugin.so" name="${prefix}mimic_robotiq_85_4">
         <joint>${prefix}finger_joint</joint>
-        <mimicJoint>${prefix}right_inner_finger_joint</mimicJoint>
+        <mimicJoint>${prefix}right_distal_phalanx_joint</mimicJoint>
         <multiplier>-1.0</multiplier>
       </plugin>
@@ -61,11 +61,11 @@
         <material>Gazebo/Grey</material>
     </gazebo>
-    <gazebo reference="${prefix}left_outer_finger">
+    <gazebo reference="${prefix}left_bar">
         <material>Gazebo/Black</material>
     </gazebo>
-    <gazebo reference="${prefix}left_inner_finger">
+    <gazebo reference="${prefix}left_distal_phalanx">
         <material>Gazebo/Grey</material>
     </gazebo>
-    <gazebo reference="${prefix}left_inner_knuckle">
+    <gazebo reference="${prefix}left_proximal_phalanx">
         <material>Gazebo/Black</material>
     </gazebo>
@@ -73,11 +73,11 @@
         <material>Gazebo/Grey</material>
     </gazebo>
-    <gazebo reference="${prefix}right_outer_finger">
+    <gazebo reference="${prefix}right_bar">
         <material>Gazebo/Black</material>
     </gazebo>
-    <gazebo reference="${prefix}right_inner_finger">
+    <gazebo reference="${prefix}right_distal_phalanx">
         <material>Gazebo/Grey</material>
     </gazebo>
-    <gazebo reference="${prefix}right_inner_knuckle">
+    <gazebo reference="${prefix}right_proximal_phalanx">
         <material>Gazebo/Black</material>
     </gazebo>

File: robotiq_2f_85_gripper_visualization/urdf/robotiq_arg2f_85_macro.xacro (robot description, xacro)
@@ -19,5 +19,5 @@
           <origin xyz="0 0 0" rpy="0 0 0" />
           <geometry>
-            <mesh filename="package://robotiq_2f_85_gripper_visualization/meshes/visual/robotiq_arg2f_85_outer_knuckle.dae" scale="0.001 0.001 0.001"/>
+            <mesh filename="package://robotiq_2f_85_gripper_visualization/meshes/visual/outer_knuckle.stl" />
           </geometry>
           <material name="">
@@ -28,11 +28,11 @@
           <origin xyz="0 0 0" rpy="0 0 0" />
           <geometry>
-            <mesh filename="package://robotiq_2f_85_gripper_visualization/meshes/collision/robotiq_arg2f_85_outer_knuckle.dae" scale="0.001 0.001 0.001"/>
-          </geometry>
-        </collision>
-      </link>
-    </xacro:macro>
-    <xacro:macro name="outer_finger" params="prefix fingerprefix">
-      <link name="${prefix}${fingerprefix}_outer_finger">
+            <mesh filename="package://robotiq_2f_85_gripper_visualization/meshes/collision/outer_knuckle.stl"/>
+          </geometry>
+        </collision>
+      </link>
+    </xacro:macro>
+    <xacro:macro name="bar" params="prefix fingerprefix">
+      <link name="${prefix}${fingerprefix}_bar">
         <inertial>
           <origin xyz="0.00030115855001899 0.0373907951953854 -0.0208027427000385" rpy="0 0 0" />
@@ -43,20 +43,20 @@
           <origin xyz="0 0 0" rpy="0 0 0" />
           <geometry>
-            <mesh filename="package://robotiq_2f_85_gripper_visualization/meshes/visual/robotiq_arg2f_85_outer_finger.dae" scale="0.001 0.001 0.001"/>
-          </geometry>
-          <material name="">
-            <color rgba="0.1 0.1 0.1 1" />
-          </material>
-        </visual>
-        <collision>
-          <origin xyz="0 0 0" rpy="0 0 0" />
-          <geometry>
-            <mesh filename="package://robotiq_2f_85_gripper_visualization/meshes/collision/robotiq_arg2f_85_outer_finger.dae" scale="0.001 0.001 0.001"/>
-          </geometry>
-        </collision>
-      </link>
-    </xacro:macro>
-    <xacro:macro name="inner_knuckle" params="prefix fingerprefix">
-      <link name="${prefix}${fingerprefix}_inner_knuckle">
+            <mesh filename="package://robotiq_2f_85_gripper_visualization/meshes/visual/bar.stl" />
+          </geometry>
+          <material name="">
+            <color rgba="0.1 0.1 0.1 1" />
+          </material>
+        </visual>
+        <collision>
+          <origin xyz="0 0 0" rpy="0 0 0" />
+          <geometry>
+            <mesh filename="package://robotiq_2f_85_gripper_visualization/meshes/collision/bar.stl" />
+          </geometry>
+        </collision>
+      </link>
+    </xacro:macro>
+    <xacro:macro name="proximal_phalanx" params="prefix fingerprefix">
+      <link name="${prefix}${fingerprefix}_proximal_phalanx">
         <inertial>
           <origin xyz="0.000123011831763771 0.0507850843201817 0.00103968640075166" rpy="0 0 0" />
@@ -67,20 +67,20 @@
           <origin xyz="0 0 0" rpy="0 0 0" />
           <geometry>
-            <mesh filename="package://robotiq_2f_85_gripper_visualization/meshes/visual/robotiq_arg2f_85_inner_knuckle.dae" scale="0.001 0.001 0.001"/>
-          </geometry>
-          <material name="">
-            <color rgba="0.1 0.1 0.1 1" />
-          </material>
-        </visual>
-        <collision>
-          <origin xyz="0 0 0" rpy="0 0 0" />
-          <geometry>
-            <mesh filename="package://robotiq_2f_85_gripper_visualization/meshes/collision/robotiq_arg2f_85_inner_knuckle.dae" scale="0.001 0.001 0.001"/>
-          </geometry>
-        </collision>
-      </link>
-    </xacro:macro>
-    <xacro:macro name="inner_finger" params="prefix fingerprefix">
-      <link name="${prefix}${fingerprefix}_inner_finger">
+            <mesh filename="package://robotiq_2f_85_gripper_visualization/meshes/visual/proximal_phalanx.stl" />
+          </geometry>
+          <material name="">
+            <color rgba="0.1 0.1 0.1 1" />
+          </material>
+        </visual>
+        <collision>
+          <origin xyz="0 0 0" rpy="0 0 0" />
+          <geometry>
+            <mesh filename="package://robotiq_2f_85_gripper_visualization/meshes/collision/proximal_phalanx.stl" />
+          </geometry>
+        </collision>
+      </link>
+    </xacro:macro>
+    <xacro:macro name="distal_phalanx" params="prefix fingerprefix">
+      <link name="${prefix}${fingerprefix}_distal_phalanx">
         <inertial>
           <origin xyz="0.000299999999999317 0.0160078233491243 -0.0136945669206257" rpy="0 0 0" />
@@ -91,14 +91,14 @@
           <origin xyz="0 0 0" rpy="0 0 0" />
           <geometry>
-            <mesh filename="package://robotiq_2f_85_gripper_visualization/meshes/visual/robotiq_arg2f_85_inner_finger.dae" scale="0.001 0.001 0.001"/>
-          </geometry>
-          <material name="">
-            <color rgba="0.1 0.1 0.1 1" />
-          </material>
-        </visual>
-        <collision>
-          <origin xyz="0 0 0" rpy="0 0 0" />
-          <geometry>
-            <mesh filename="package://robotiq_2f_85_gripper_visualization/meshes/collision/robotiq_arg2f_85_inner_finger.dae" scale="0.001 0.001 0.001" />
+            <mesh filename="package://robotiq_2f_85_gripper_visualization/meshes/visual/distal_phalanx.stl" />
+          </geometry>
+          <material name="">
+            <color rgba="0.1 0.1 0.1 1" />
+          </material>
+        </visual>
+        <collision>
+          <origin xyz="0 0 0" rpy="0 0 0" />
+          <geometry>
+            <mesh filename="package://robotiq_2f_85_gripper_visualization/meshes/collision/distal_phalanx.stl" />
           </geometry>
         </collision>
@@ -106,6 +106,6 @@
     </xacro:macro>
     <!-- Finger pad link, the default are the "big pads" with rubber-->
-    <xacro:macro name="inner_finger_pad" params="prefix fingerprefix">
-      <link name="${prefix}${fingerprefix}_inner_finger_pad">
+    <!-- <xacro:macro name="pad" params="prefix fingerprefix">
+      <link name="${prefix}${fingerprefix}_pad">
         <visual>
           <origin xyz="0 0 0" rpy="0 0 0" />
@@ -127,27 +127,26 @@
         </collision>
       </link>
-    </xacro:macro>
+    </xacro:macro> -->
     <xacro:macro name="finger_links" params="prefix fingerprefix">
       <xacro:outer_knuckle prefix="${prefix}" fingerprefix="${fingerprefix}"/>
-      <xacro:outer_finger prefix="${prefix}" fingerprefix="${fingerprefix}"/>
-      <xacro:inner_finger prefix="${prefix}" fingerprefix="${fingerprefix}"/>
-      <xacro:inner_finger_pad prefix="${prefix}" fingerprefix="${fingerprefix}"/>
-      <xacro:inner_knuckle prefix="${prefix}" fingerprefix="${fingerprefix}"/>
+      <xacro:bar prefix="${prefix}" fingerprefix="${fingerprefix}"/>
+      <xacro:distal_phalanx prefix="${prefix}" fingerprefix="${fingerprefix}"/>
+      <!-- <xacro:pad prefix="${prefix}" fingerprefix="${fingerprefix}"/> -->
+      <xacro:proximal_phalanx prefix="${prefix}" fingerprefix="${fingerprefix}"/>
     </xacro:macro>
     <!-- fingers joints macros -->
-    <xacro:macro name="outer_finger_joint" params="prefix fingerprefix">
-      <joint name="${prefix}${fingerprefix}_outer_finger_joint" type="fixed">
+    <xacro:macro name="bar_joint" params="prefix fingerprefix">
+      <joint name="${prefix}${fingerprefix}_bar_joint" type="fixed">
         <origin xyz="0 0.0315 -0.0041" rpy="0 0 0"/>
         <parent link="${prefix}${fingerprefix}_outer_knuckle" />
-        <child link="${prefix}${fingerprefix}_outer_finger" />
+        <child link="${prefix}${fingerprefix}_bar" />
         <axis xyz="1 0 0" />
       </joint>
     </xacro:macro>
-    <xacro:macro name="inner_knuckle_joint" params="prefix fingerprefix reflect">
-      <joint name="${prefix}${fingerprefix}_inner_knuckle_joint" type="revolute">
-        <!-- <origin xyz="0 ${reflect * -0.0127} 0.06142" rpy="${pi / 2 + .725} 0 ${(reflect - 1) * pi / 2}" /> -->
-        <origin xyz="0 ${reflect * -0.0127} 0.06142" rpy="0 0 ${(1 + reflect) * pi / 2}"/>
+    <xacro:macro name="proximal_phalanx_joint" params="prefix fingerprefix reflect">
+      <joint name="${prefix}${fingerprefix}_proximal_phalanx_joint" type="revolute">
+        <origin xyz="0 ${reflect * -0.0127} 0.06142" rpy=".125 0 ${(1 + reflect) * pi / 2}"/>
         <parent link="${prefix}robotiq_arg2f_base_link" />
-        <child link="${prefix}${fingerprefix}_inner_knuckle" />
+        <child link="${prefix}${fingerprefix}_proximal_phalanx" />
         <axis xyz="1 0 0" />
         <limit lower="0" upper="0.8757" velocity="0.5" effort="1000" />
@@ -155,9 +154,9 @@
       </joint>
     </xacro:macro>
-    <xacro:macro name="inner_finger_joint" params="prefix fingerprefix">
-      <joint name="${prefix}${fingerprefix}_inner_finger_joint" type="revolute">
+    <xacro:macro name="distal_phalanx_joint" params="prefix fingerprefix">
+      <joint name="${prefix}${fingerprefix}_distal_phalanx_joint" type="revolute">
         <origin xyz="0 0.0061 0.0471" rpy="0 0 0"/>
-        <parent link="${prefix}${fingerprefix}_outer_finger" />
-        <child link="${prefix}${fingerprefix}_inner_finger" />
+        <parent link="${prefix}${fingerprefix}_bar" />
+        <child link="${prefix}${fingerprefix}_distal_phalanx" />
         <axis xyz="1 0 0" />
         <limit lower="-0.8757" upper="0" velocity="0.5" effort="1000" />
@@ -165,17 +164,17 @@
       </joint>
     </xacro:macro>
-    <xacro:macro name="inner_finger_pad_joint" params="prefix fingerprefix">
-      <joint name="${prefix}${fingerprefix}_inner_finger_pad_joint" type="fixed">
+    <!-- <xacro:macro name="pad_joint" params="prefix fingerprefix">
+      <joint name="${prefix}${fingerprefix}_pad_joint" type="fixed">
         <origin xyz="0 -0.0220203446692936 0.03242" rpy="0 0 0"/>
-        <parent link="${prefix}${fingerprefix}_inner_finger" />
-        <child link="${prefix}${fingerprefix}_inner_finger_pad" />
+        <parent link="${prefix}${fingerprefix}_distal_phalanx" />
+        <child link="${prefix}${fingerprefix}_pad" />
         <axis xyz="0 0 1" />
       </joint>
-    </xacro:macro>
+    </xacro:macro> -->
     <xacro:macro name="finger_joints" params="prefix fingerprefix reflect">
-      <xacro:outer_finger_joint prefix="${prefix}" fingerprefix="${fingerprefix}"/>
-      <xacro:inner_knuckle_joint prefix="${prefix}" fingerprefix="${fingerprefix}" reflect="${reflect}"/>
-      <xacro:inner_finger_joint prefix="${prefix}" fingerprefix="${fingerprefix}"/>
-      <xacro:inner_finger_pad_joint prefix="${prefix}" fingerprefix="${fingerprefix}"/>
+      <xacro:bar_joint prefix="${prefix}" fingerprefix="${fingerprefix}"/>
+      <xacro:proximal_phalanx_joint prefix="${prefix}" fingerprefix="${fingerprefix}" reflect="${reflect}"/>
+      <xacro:distal_phalanx_joint prefix="${prefix}" fingerprefix="${fingerprefix}"/>
+      <!-- <xacro:pad_joint prefix="${prefix}" fingerprefix="${fingerprefix}"/> -->
     </xacro:macro>
     <!-- base link -->
@@ -188,5 +187,5 @@
         <inertial>
           <origin xyz="8.625E-08 -4.6583E-06 0.03145" rpy="0 0 0" />
-          <mass value="0.22652" />
+          <mass value="0.7" />
           <inertia ixx="0.00020005" ixy="-4.2442E-10" ixz="-2.9069E-10" iyy="0.00017832" iyz="-3.4402E-08" izz="0.00013478" />
         </inertial>
@@ -194,14 +193,14 @@
           <origin xyz="0 0 0" rpy="0 0 0" />
           <geometry>
-            <mesh filename="package://robotiq_2f_85_gripper_visualization/meshes/visual/robotiq_arg2f_base_link.stl" />
-          </geometry>
-          <material name="">
-            <color rgba="0.1 0.1 0.1 1" />
-          </material>
-        </visual>
-        <collision>
-          <origin xyz="0 0 0" rpy="0 0 0" />
-          <geometry>
-            <mesh filename="package://robotiq_2f_85_gripper_visualization/meshes/collision/robotiq_arg2f_base_link.stl" />
+            <mesh filename="package://robotiq_2f_85_gripper_visualization/meshes/visual/base_link.dae" />
+          </geometry>
+          <material name="">
+            <color rgba="0.1 0.1 0.1 1" />
+          </material>
+        </visual>
+        <collision>
+          <origin xyz="0 0 0" rpy="0 0 0" />
+          <geometry>
+            <mesh filename="package://robotiq_2f_85_gripper_visualization/meshes/collision/base_link.stl" />
           </geometry>
         </collision>
