Commit message: Modifications doen for correct representation of the robotiq gripper in urdf

File: robotiq_epick_visualization/urdf/robotiq_epick_model_macro.xacro (robot description, xacro)
@@ -12,5 +12,5 @@
       </inertial>
       <visual>
-        <origin xyz="0 0 ${0.097/2}" rpy="0 0 0"/>
+        <origin xyz="0 0 ${0.097/2}" rpy="0 0 ${.5 * pi}"/>
         <geometry>
           <mesh filename="package://robotiq_epick_visualization/meshes/visual/robotiq_epick.dae" scale="0.001 0.001 0.001"/>
@@ -21,5 +21,5 @@
       </visual>
       <visual>
-        <origin xyz="0 0 ${0.08/2+0.097}" rpy="0 0 0"/>
+        <origin xyz="0 0 ${0.1}" rpy="0 0 0"/>
         <geometry>
           <cylinder radius="0.006" length="0.08"/>
@@ -38,11 +38,11 @@
       <collision>
         <!-- -0.095 + 0.102/2 = -0.044-->
-        <origin xyz="0 0 ${0.114/2}" rpy="0 0 0"/>
+        <origin xyz="0 0 0" rpy="0 0 0"/>
         <geometry>
-          <cylinder radius="0.035" length="0.114"/>
+          <cylinder radius="0.05" length="0.12"/>
         </geometry>
       </collision>
       <collision>
-        <origin xyz="0 0 ${0.08/2+0.097}" rpy="0 0 0"/>
+        <origin xyz="0 0 ${0.1}" rpy="0 0 0"/>
         <geometry>
           <cylinder radius="0.006" length="0.08"/>
@@ -68,5 +68,5 @@
       <gravity>0</gravity>
       <visual>
-        <origin rpy="0 0 0" xyz="0 0 .005"/>
+        <origin rpy="0 0 0" xyz="0 0 -.04"/>
         <geometry>
           <cylinder radius="0.0225" length="0.01"/>
@@ -77,5 +77,5 @@
       </visual>
       <collision>
-        <origin rpy="0 0 0" xyz="0 0 .005"/>
+        <origin rpy="0 0 0" xyz="0 0 -0.04"/>
         <geometry>
           <cylinder radius="0.0225" length="0.01"/>

Commit message: Increase epick rod length to match reality

File: robotiq_epick_visualization/urdf/robotiq_epick_model_macro.xacro (robot description, xacro)
@@ -40,9 +40,9 @@
         <origin xyz="0 0 0" rpy="0 0 0"/>
         <geometry>
-          <cylinder radius="0.05" length="0.12"/>
+          <cylinder radius="0.05" length="0.18"/>
         </geometry>
       </collision>
       <collision>
-        <origin xyz="0 0 ${0.1}" rpy="0 0 0"/>
+        <origin xyz="0 0 ${0.12}" rpy="0 0 0"/>
         <geometry>
           <cylinder radius="0.006" length="0.08"/>
@@ -63,5 +63,5 @@
       <parent link="${hand_link_name}"/>
       <child link="epick_end_effector"/>
-      <origin xyz="0 0 ${.097+.090}" rpy="0 0 0"/>
+      <origin xyz="0 0 ${.12+.090}" rpy="0 0 0"/>
     </joint>
     <link name="epick_end_effector">

Commit message: Better aligning visual and collision models

File: robotiq_epick_visualization/urdf/robotiq_epick_model_macro.xacro (robot description, xacro)
@@ -21,7 +21,7 @@
       </visual>
       <visual>
-        <origin xyz="0 0 ${0.1}" rpy="0 0 0"/>
+        <origin xyz="0 0 ${0.12}" rpy="0 0 0"/>
         <geometry>
-          <cylinder radius="0.006" length="0.08"/>
+          <cylinder radius="0.006" length="0.12"/>
         </geometry>
         <material name="mat2">
@@ -29,22 +29,8 @@
         </material>
       </visual>
-        <!-- -0.095 + 0.102/2 = -0.044-->
-      <!-- <visual>
-        <origin xyz="0 0 ${-0.044+0.095+0.014+0.09}" rpy="0 0 0"/>
-        <geometry>
-          <cylinder radius="0.006" length="0.09"/>
-        </geometry>
-      </visual>  -->
-      <collision>
-        <!-- -0.095 + 0.102/2 = -0.044-->
-        <origin xyz="0 0 0" rpy="0 0 0"/>
-        <geometry>
-          <cylinder radius="0.05" length="0.18"/>
-        </geometry>
-      </collision>
       <collision>
         <origin xyz="0 0 ${0.12}" rpy="0 0 0"/>
         <geometry>
-          <cylinder radius="0.006" length="0.08"/>
+          <cylinder radius="0.006" length="0.12"/>
         </geometry>
         <material name="mat2">
@@ -52,4 +38,10 @@
         </material>
       </collision>
+      <!-- <collision>
+        <origin xyz="0 0 0" rpy="0 0 0"/>
+        <geometry>
+          <cylinder radius="0.05" length="0.08"/>
+        </geometry>
+      </collision> -->
       <!-- -0.095 + 0.102/2 = -0.044-->
       <!-- <collision>
@@ -63,5 +55,5 @@
       <parent link="${hand_link_name}"/>
       <child link="epick_end_effector"/>
-      <origin xyz="0 0 ${.12+.090}" rpy="0 0 0"/>
+      <origin xyz="0 0 ${.15+.090}" rpy="0 0 0"/>
     </joint>
     <link name="epick_end_effector">
