Commit message: Phase 0 archive: emmons:/home/aurmr/workspaces/capacitive_cup/src/aurmr_tahoma/third-party/robotiq
Branch: DETACHED
Base HEAD: c0140b90a7e5c4f802e9310c6b1fccbdcadf2df5
Includes uncommitted tracked changes and untracked code/config.
Excluded untracked files (noise/data/>5MB): 0

File: robotiq_epick_visualization/urdf/robotiq_epick_model_macro.xacro (robot description, xacro)
@@ -37,11 +37,26 @@
       </visual>  -->
       <collision>
-        <!-- -0.095 + 0.102/2 = -0.044-->
-        <origin xyz="0 0 0" rpy="0 0 0"/>
+        <!-- 0.107 / 2 = 0.0535 -->
+        <origin xyz="0 0 0.0535" rpy="0 0 0"/>
         <geometry>
-          <cylinder radius="0.05" length="0.12"/>
+          <cylinder radius="0.06" length="0.107"/>
         </geometry>
       </collision>
       <collision>
+        <!-- 0.107 + 0.006 / 2 = 0.110-->
+        <origin xyz="0 ${0.04} 0.110" rpy="0 0 0"/>
+        <geometry>
+          <box size = "0.052 0.08 0.006"/>
+        </geometry>
+      </collision>
+      <collision>
+      <!-- 0.107 + 0.078 / 2 = 0.146-->
+        <origin xyz="0 0 ${0.146}" rpy="0 0 0"/>
+        <geometry>
+          <cylinder radius="0.06" length="0.078"/>
+        </geometry>
+      </collision>
+      <!-- Previous single finger pipe nipple-->
+      <!-- <collision>
         <origin xyz="0 0 ${0.1}" rpy="0 0 0"/>
         <geometry>
@@ -51,12 +66,6 @@
           <color rgba="1 0 0 1"/>
         </material>
-      </collision>
-      <!-- -0.095 + 0.102/2 = -0.044-->
-      <!-- <collision>
-        <origin xyz="0 0 ${-0.044+0.095+0.014+0.09}" rpy="0 0 0"/>
-        <geometry>
-          <cylinder radius="0.006" length="0.09"/>
-        </geometry>
-      </collision>     -->
+      </collision> -->
+      <!-- Previous single finger pipe nipple-->
     </link>
     <joint name="$hand__end_effector_joint" type="fixed">

Commit message: Phase 0 archive: emmons:/home/aurmr/workspaces/markus_test/src/aurmr_tahoma/third-party/robotiq
Branch: henri-continual
Base HEAD: 30ffbfc1722a101abab034a6ce915132f6a246f5
Includes uncommitted tracked changes and untracked code/config.
Excluded untracked files (noise/data/>5MB): 0

File: robotiq_epick_visualization/urdf/robotiq_epick_model_macro.xacro (robot description, xacro)
@@ -32,5 +32,5 @@
         <origin xyz="0 0 ${0.12}" rpy="0 0 0"/>
         <geometry>
-          <cylinder radius="0.006" length="0.12"/>
+          <cylinder radius="0.0375" length="0.195"/>
         </geometry>
         <material name="mat2">
